Commit message: finial_backup

File: robot_simulation/urdf/robot.xacro (robot description, xacro)
@@ -11,5 +11,5 @@
   <xacro:include filename="$(find robot_simulation)/urdf/materials.xacro" />
   <xacro:include filename="$(find robot_simulation)/urdf/xbot-u.urdf.xacro" />
-  <xacro:include filename="$(find robot_simulation)/urdf/xbot-u.gazebo" />
+  <!-- <xacro:include filename="$(find robot_simulation)/urdf/xbot-u.gazebo" /> -->
   <xacro:xbot2_base/>
 </robot>

File: robot_simulation/urdf/sick_tim.urdf.xacro (robot description, xacro)
@@ -57,75 +57,43 @@
       </inertial>
     </link>
-    <xacro:sick_tim_laser_gazebo_v0 name="${name}" link="${name}" ros_topic="${ros_topic}"
-    update_rate="15.0" min_angle="-2.357" max_angle="2.357" min_range="${min_range}" max_range="${max_range}"/>
-    <!--update_rate=15.0-->
+      <xacro:sick_tim_laser_gazebo_v0 name="${name}" link="${name}" ros_topic="${ros_topic}"
+      update_rate="15.0" min_angle="-2.357" max_angle="2.357" min_range="${min_range}" max_range="${max_range}"/>
+      <!--update_rate=15.0-->
   </xacro:macro>
   <xacro:macro name="sick_tim_laser_gazebo_v0" params="name link ros_topic update_rate min_angle max_angle min_range max_range">
-    <!--gazebo reference="${link}">
-      <material value="Gazebo/LightWood" />
-      <sensor type="gpu_ray" name="${name}">
-      <sensor type="ray" name="${name}">
+    <gazebo reference="${link}">
+      <sensor type="gpu_lidar" name="${name}">
+        <pose>0 0 0 0 0 0</pose>
+        <visualize>true</visualize>
+        <update_rate>20.0</update_rate>
+        <!-- <topic>scan</topic> -->
+        <topic>${ros_topic}</topic>
+        <gz_frame_id>${link}</gz_frame_id>
         <always_on>true</always_on>
-        <update_rate>${update_rate}</update_rate>
-        <pose>0 0 0 0 0 0</pose>
-        <visualize>false</visualize>
-        <ray>
+        <lidar>
           <scan>
             <horizontal>
+              <!-- <samples>1080</samples> -->
               <samples>810</samples>
-              <resolution>1</resolution>
-              <min_angle>${min_angle}</min_angle>
-              <max_angle>${max_angle}</max_angle>
+              <resolution>1.000000</resolution>
+              <min_angle>-1.570796</min_angle>
+              <max_angle>1.570796</max_angle>
+              <!-- <min_angle>-3.14159265</min_angle>
+              <max_angle>3.14159265</max_angle> -->
             </horizontal>
           </scan>
           <range>
-            <min>${min_range}</min>
-            <max>${max_range}</max>
+            <min>0.10</min>
+            <max>10.0</max>
             <resolution>0.01</resolution>
           </range>
-        </ray>
-        <plugin name="gazebo_ros_${name}_controller" filename="libgazebo_ros_gpu_laser.so">
-        <!plugin name="gazebo_ros_${name}_controller" filename="libgazebo_ros_laser.so" >
-          <gaussianNoise>0.01</gaussianNoise>
-          <alwaysOn>true</alwaysOn>
-          <updateRate>${update_rate}</updateRate>
-          <topicName>${ros_topic}</topicName>
-          <frameName>${link}</frameName>
-        </plugin>
+          <noise>
+            <type>gaussian</type>
+            <mean>0.0</mean>
+            <stddev>0.01</stddev>
+          </noise>
+        </lidar>
       </sensor>
-    </gazebo-->
-  <gazebo reference="${link}">
-    <sensor type="gpu_lidar" name="${name}">
-      <pose>0 0 0 0 0 0</pose>
-      <visualize>true</visualize>
-      <update_rate>${update_rate}</update_rate>
-      <!-- <topic>scan</topic> -->
-      <topic>${ros_topic}</topic>
-      <gz_frame_id>${link}</gz_frame_id>
-      <always_on>true</always_on>
-      <lidar>
-        <scan>
-          <horizontal>
-            <samples>810</samples>
-            <resolution>1</resolution>
-            <min_angle>-1.570796</min_angle>
-            <max_angle>1.570796</max_angle>
-          </horizontal>
-        </scan>
-        <range>
-          <min>0.10</min>
-          <max>10.0</max>
-          <resolution>0.01</resolution>
-        </range>
-        <noise>
-          <type>gaussian</type>
-          <mean>0.0</mean>
-          <stddev>0.01</stddev>
-        </noise>
-        <!-- <topicName>${ros_topic}</topicName>
-        <frameName>${link}</frameName> -->
-      </lidar>
-    </sensor>
-  </gazebo>
+    </gazebo>
   </xacro:macro>
 </robot>

File: robot_simulation/urdf/xbot-u.urdf.xacro (robot description, xacro)
@@ -99,5 +99,5 @@
     <parent link="base_link"/>
     <child link="left_wheel"/>
-    <limit effort="6" velocity="1.0"/>
+    <limit effort="6" velocity="5.0"/>
     <joint_properties damping="0.0" friction="0.0"/>
   </joint>
@@ -126,5 +126,5 @@
     <parent link="base_link"/>
     <child link="right_wheel"/>
-    <limit effort="6" velocity="1.0"/>
+    <limit effort="6" velocity="5.0"/>
     <joint_properties damping="0.0" friction="0.0"/>
   </joint>
@@ -221,4 +221,186 @@
   <link name="camera_link_optical">
   </link>
+  <transmission name="tran1">
+    <type>transmission_interface/SimpleTransmission</type>
+    <joint name="base_to_yaw_platform">
+      <hardwareInterface>EffortJointInterface</hardwareInterface>
+    </joint>
+    <actuator name="yaw_motor">
+      <hardwareInterface>EffortJointInterface</hardwareInterface>
+      <mechanicalReduction>1</mechanicalReduction>
+    </actuator>
+  </transmission>
+  <transmission name="tran2">
+    <type>transmission_interface/SimpleTransmission</type>
+    <joint name="yaw_to_pitch_platform">
+      <hardwareInterface>EffortJointInterface</hardwareInterface>
+    </joint>
+    <actuator name="pitch_motor">
+      <hardwareInterface>EffortJointInterface</hardwareInterface>
+      <mechanicalReduction>1</mechanicalReduction>
+    </actuator>
+  </transmission>
+   <ros2_control name="GazeboSimSystem" type="system">
+    <hardware>
+      <plugin>gz_ros2_control/GazeboSimSystem</plugin>
+    </hardware>
+    <joint name="base_to_yaw_platform">
+      <command_interface name="effort"/>
+      <!-- <state_interface name="position"/>
+      <state_interface name="velocity"/> -->
+      <state_interface name="effort"/>
+    </joint>
+    <joint name="yaw_to_pitch_platform">
+      <command_interface name="effort"/>
+      <!-- <state_interface name="position"/>
+      <state_interface name="velocity"/> -->
+      <state_interface name="effort"/>
+    </joint>
+  </ros2_control>
+  <gazebo>
+    <plugin filename="libgz_ros2_control-system" name="gz_ros2_control::GazeboSimROS2ControlPlugin">
+      <parameters>$(find robot_simulation)/param/xbot-u_control.yaml</parameters>
+      <robot_param>robot_description</robot_param>
+      <robot_param_node>robot_state_publisher</robot_param_node>
+      <controller_manager_prefix_node_name>controller_manager</controller_manager_prefix_node_name>
+    </plugin>
+  </gazebo>
+  <gazebo reference="imu_link">
+    <sensor name="imu_sensor" type="imu">
+      <always_on>true</always_on>
+      <update_rate>100</update_rate>
+      <visualize>true</visualize>
+      <topic>imu</topic>
+      <imu>
+        <angular_velocity>
+            <x>
+              <noise type="gaussian">
+                <mean>0.0</mean>
+                <stddev>2e-4</stddev>
+              </noise>
+            </x>
+            <y>
+              <noise type="gaussian">
+                <mean>0.0</mean>
+                <stddev>2e-4</stddev>
+              </noise>
+            </y>
+            <z>
+              <noise type="gaussian">
+                <mean>0.0</mean>
+                <stddev>2e-4</stddev>
+              </noise>
+            </z>
+          </angular_velocity>
+          <linear_acceleration>
+            <x>
+              <noise type="gaussian">
+                <mean>0.0</mean>
+                <stddev>1.7e-2</stddev>
+              </noise>
+            </x>
+            <y>
+              <noise type="gaussian">
+                <mean>0.0</mean>
+                <stddev>1.7e-2</stddev>
+              </noise>
+            </y>
+            <z>
+              <noise type="gaussian">
+                <mean>0.0</mean>
+                <stddev>1.7e-2</stddev>
+              </noise>
+            </z>
+          </linear_acceleration>
+      </imu>
+    </sensor>
+  </gazebo>
+  <gazebo reference="camera_link">
+    <sensor type="rgbd_camera" name="camera_D415_point">
+      <updateRate>30.0</updateRate>
+      <alwaysOn>true</alwaysOn>
+      <visualize>true</visualize>
+      <topic>camera/depth</topic>
+      <gz_frame_id>camera_link</gz_frame_id>
+      <camera name="head">
+        <horizontal_fov>1.05</horizontal_fov>
+        <image>
+          <width>1280</width>
+          <height>720</height>
+          <format>R8G8B8</format>
+        </image>
+        <clip>
+          <near>0.1</near>
+          <far>10.0</far>
+        </clip>
+        <noise>
+          <type>gaussian</type>
+          <mean>0.0</mean>
+          <stddev>0.005</stddev>
+        </noise>
+        <baseline>0.1</baseline>
+        <distortion_k1>0.0</distortion_k1>
+        <distortion_k2>0.0</distortion_k2>
+        <distortion_k3>0.0</distortion_k3>
+        <distortion_t1>0.0</distortion_t1>
+        <distortion_t2>0.0</distortion_t2>
+        <pointCloudCutoff>0.05</pointCloudCutoff>
+        <rangeMax>4.0</rangeMax>
+      </camera>
+    </sensor>
+  </gazebo>
+  <gazebo>
+    <plugin filename="gz-sim-diff-drive-system" name="gz::sim::systems::DiffDrive">
+        <odom_topic>odom</odom_topic>
+        <frame_id>odom</frame_id>
+        <topic>cmd_vel</topic>
+        <alwaysOn>true</alwaysOn>
+        <odom_publisher_frequency>20</odom_publisher_frequency>
+        <left_joint>left_wheel_hinge</left_joint>
+        <right_joint>right_wheel_hinge</right_joint>
+        <wheel_separation>0.46</wheel_separation>
+        <wheel_radius>0.19</wheel_radius>
+        <tf_topic>/tf_diff</tf_topic>
+        <child_frame_id>base_footprint</child_frame_id>
+    </plugin>
+  </gazebo>
+  <gazebo reference="base_link">
+    <mu>0</mu>
+    <mu2>0</mu2>
+    <kp>100000000.0</kp>
+    <kd>10000.0</kd>
+  </gazebo>
+  <gazebo reference="laser">
+  </gazebo>
+  <gazebo reference="right_wheel">
+    <mu>10</mu>
+    <mu2>10</mu2>
+    <kp>100.0</kp>
+    <kd>10.0</kd>
+  </gazebo>
+  <gazebo reference="left_wheel">
+    <mu>10</mu>
+    <mu2>10</mu2>
+    <kp>100.0</kp>
+    <kd>10.0</kd>
+  </gazebo>
+  <gazebo reference="yaw_platform">
+    <mu>.5</mu>
+    <mu2>.5</mu2>
+  </gazebo>
+  <gazebo reference="pitch_platform">
+    <mu>.5</mu>
+    <mu2>.5</mu2>
+  </gazebo>
+  <gazebo>
+    <plugin filename="gz-sim-joint-state-publisher-system" name="gz::sim::systems::JointStatePublisher">
+        <topic>joint_states</topic>
+        <!-- <update_rate>30</update_rate> -->
+        <joint_name>left_wheel_hinge</joint_name>
+        <joint_name>right_wheel_hinge</joint_name>
+        <joint_name>base_to_yaw_platform</joint_name>
+        <joint_name>yaw_to_pitch_platform</joint_name>
+    </plugin>
+  </gazebo>
   </xacro:macro>
 </robot>
